File: 2607363-Felipe Ferrero-Microduino/2607363-Felipe Ferrero-Microduino.kicad_pcb (KiCad board)
At the start: 2 copper layers, 14 parts, among them J1 USB_A, J2 Header, U1 ATtiny85-20S

Commit message: Mi prrimer commit y entrga de protecto de kicad
Other:
- board outline added: 30.5 x 28.5 mm
Changed lines of the file:
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@@
 		(at 156 113.5)
 		(property "Reference" "D4"
-			(at -2.6 2.725 0)
+			(at -0.5 2 0)
 			(layer "F.SilkS")
 			(effects
@@
 			(type default)
 		)
-		(layer "F.Cu")
+		(layer "Edge.Cuts")
 	)
 	(gr_line
@@
 			(type default)
 		)
-		(layer "F.Cu")
+		(layer "Edge.Cuts")
 	)
 	(gr_line
@@
 			(type default)
 		)
-		(layer "F.Cu")
+		(layer "Edge.Cuts")
 	)
 	(gr_line
@@
 			(type default)
 		)
-		(layer "F.Cu")
+		(layer "Edge.Cuts")
 	)
 	(gr_line
@@
 			(type default)
 		)
-		(layer "F.Cu")
+		(layer "Edge.Cuts")
 	)
 	(gr_line
@@
 			(type default)
 		)
-		(layer "F.Cu")
+		(layer "Edge.Cuts")
 	)
 	(gr_line
@@
 			(type default)
 		)
-		(layer "F.Cu")
+		(layer "Edge.Cuts")
 	)
 	(gr_line
@@
 			(type default)
 		)
-		(layer "F.Cu")
-	)
-	(gr_line
+		(layer "Edge.Cuts")
+	)
+	(gr_line

Commit message: Actualización Microduino
Routing:
- net GND: track 66.1 -> 100.0 mm
Changed lines of the file:
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@@
+	)
+	(segment
+		(start 169.360559 122.5)
+		(end 151 122.5)
+		(width 0.6)
+		(layer "F.Cu")
+		(net "GND")
+	)
+	(segment
+		(start 170.97 114.303631)
+		(end 170.97 120.890559)
+		(width 0.6)
+		(layer "F.Cu")
+		(net "GND")
 	)
 	(segment
@@
 	)
 	(segment
+		(start 168.5875 112.595)
+		(end 169.261369 112.595)
+		(width 0.6)
+		(layer "F.Cu")
+		(net "GND")
+	)
+	(segment
 		(start 164.867588 104.5)
 		(end 165.65 105.282412)
@@
 	)
 	(segment
+		(start 169.261369 112.595)
+		(end 170.97 114.303631)
+		(width 0.6)
+		(layer "F.Cu")
+		(net "GND")
+	)
+	(segment
 		(start 166.095 112.595)
 		(end 168.5875 112.595)
@@
 	)
 	(segment
+		(start 170.97 120.890559)
+		(end 169.360559 122.5)
+		(width 0.6)
+		(layer "F.Cu")
+		(net "GND")
+	)
+	(segment
 		(start 151 104)
 		(end 151.5 104.5)
@@
 	)
 	(segment
+		(start 151 122.5)
+		(end 148.5 120)
+		(width 0.6)
+		(layer "F.Cu")
+		(net "GND")
+	)
+	(segment
 		(start 148.3 112.3)
 		(end 150 114)
@@
 	)
 	(segment
+		(start 168.5875 113.865)
+		(end 169.399999 113.865)
+		(width 0.6)
+		(layer "F.Cu")
+		(net "Net-(J2-Pin_8)")
+	)
+	(segment
 		(start 164.5 106)
 		(end 164.5 112.13137)
@@
 	)
 	(segment
-		(start 170.5 114.965001)
-		(end 169.399999 113.865)
+		(start 170.17 114.635001)
+		(end 170.17 120.559189)
+		(width 0.6)
+		(layer "F.Cu")
+		(net "Net-(J2-Pin_8)")
+	)
+	(segment
+		(start 169.379189 121.35)
+		(end 165.09 121.35)
+		(width 0.6)
+		(layer "F.Cu")
+		(net "Net-(J2-Pin_8)")
+	)
+	(segment
+		(start 169.399999 113.865)
+		(end 170.17 114.635001)
 		(width 0.6)
 		(layer "F.Cu")
@@
 	(segment
 		(start 165.09 121.35)
-		(end 169.379189 121.35)
-		(width 0.6)
-		(layer "F.Cu")
-		(net "Net-(J2-Pin_8)")
-	)
-	(segment
-		(start 169.379189 121.35)
-		(end 170.5 120.229189)
-		(width 0.6)
-		(layer "F.Cu")
-		(net "Net-(J2-Pin_8)")
-	)
-	(segment
-		(start 170.5 120.229189)
-		(end 170.5 114.965001)
+		(end 163.74 120)
 		(width 0.6)
 		(layer "F.Cu")
@@
 	)
 	(segment
-		(start 169.399999 113.865)
-		(end 168.5875 113.865)
-		(width 0.6)
-		(layer "F.Cu")
-		(net "Net-(J2-Pin_8)")
-	)
-	(segment
-		(start 163.74 120)
-		(end 165.09 121.35)
-		(width 0.6)
-		(layer "F.Cu")
+		(start 170.17 120.559189)
+		(end 169.379189 121.35)
+		(width 0.6)
+		(layer "F.Cu")
